File: Stops.sch (KiCad schematic (older format))
At the start: 19 parts

Commit message: Converted to Local and Hierarchical net labels
Parts:
- gave numbers to parts that had none: 16
Connections:
- net ESTOP_Pin: now also U5.5, U5.8; no longer U5.1, U5.2
- net SHDN_Pin: now also U5.4; no longer U5.2
- net ~ESTOP~_Pin: now also U5.6; no longer U5.2
- net at R18.1: now also U5.3; no longer U5.1
- net at R19.1: now also U5.9; no longer U5.1
Changed lines of the file:
@@
 $EndDescr
 $Comp
-L R R?
+L R R18
 U 1 1 563C0D01
 P 1550 5100
-F 0 "R?" V 1630 5100 40  0000 C CNN
+F 0 "R18" V 1630 5100 40  0000 C CNN
 F 1 "10K" V 1557 5101 40  0000 C CNN
 F 2 "~" V 1480 5100 30  0000 C CNN
@@
 $EndComp
 $Comp
-L DIODE D?
+L DIODE D2
 U 1 1 563C0D02
 P 2100 3800
-F 0 "D?" H 2100 3900 40  0000 C CNN
+F 0 "D2" H 2100 3900 40  0000 C CNN
 F 1 "DIODE" H 2100 3700 40  0000 C CNN
 F 2 "~" H 2100 3800 60  0000 C CNN
@@
 $EndComp
 $Comp
-L C C?
+L C C7
 U 1 1 563C0D03
 P 1500 3700
-F 0 "C?" H 1500 3800 40  0000 L CNN
+F 0 "C7" H 1500 3800 40  0000 L CNN
 F 1 "10uF" H 1506 3615 40  0000 L CNN
 F 2 "~" H 1538 3550 30  0000 C CNN
@@
 $EndComp
 $Comp
-L GND #PWR?
+L GND #PWR31
 U 1 1 563C0D04
 P 2100 4100
-F 0 "#PWR?" H 2100 4100 30  0001 C CNN
+F 0 "#PWR31" H 2100 4100 30  0001 C CNN
 F 1 "GND" H 2100 4030 30  0001 C CNN
 F 2 "" H 2100 4100 60  0000 C CNN
@@
 $EndComp
 $Comp
-L DIODE D?
+L DIODE D1
 U 1 1 563C0D05
 P 1800 3500
-F 0 "D?" H 1800 3600 40  0000 C CNN
+F 0 "D1" H 1800 3600 40  0000 C CNN
 F 1 "DIODE" H 1800 3400 40  0000 C CNN
 F 2 "~" H 1800 3500 60  0000 C CNN
@@
 $EndComp
 $Comp
-L NPN Q?
+L NPN Q10
 U 1 1 563C0D06
 P 1100 3500
-F 0 "Q?" H 1100 3350 50  0000 R CNN
+F 0 "Q10" H 1100 3350 50  0000 R CNN
 F 1 "NPN" H 1100 3650 50  0000 R CNN
 F 2 "~" H 1100 3500 60  0000 C CNN
@@
 	1300 3500 1600 3500
 $Comp
-L C C?
+L C C8
 U 1 1 563C0D07
 P 2300 3500
-F 0 "C?" H 2300 3600 40  0000 L CNN
+F 0 "C8" H 2300 3600 40  0000 L CNN
 F 1 "1uF" H 2306 3415 40  0000 L CNN
 F 2 "~" H 2338 3350 30  0000 C CNN
@@
 	2100 3600 2100 3500
 $Comp
-L R R?
+L R R20
 U 1 1 563C0D08
 P 1750 3300
-F 0 "R?" V 1830 3300 40  0000 C CNN
+F 0 "R20" V 1830 3300 40  0000 C CNN
 F 1 "10K" V 1757 3301 40  0000 C CNN
 F 2 "~" V 1680 3300 30  0000 C CNN
@@
 $EndComp
 $Comp
-L +5V #PWR?
+L +5V #PWR30
 U 1 1 563C0D09
 P 2000 3200
-F 0 "#PWR?" H 2000 3290 20  0001 C CNN
+F 0 "#PWR30" H 2000 3290 20  0001 C CNN
 F 1 "+5V" H 2000 3290 30  0000 C CNN
 F 2 "" H 2000 3200 60  0000 C CNN
@@
 	1000 3700 1000 4000
 Connection ~ 1500 4000
-Text GLabel 1000 3100 2    60   Input ~ 0
-WATCHDOG
 Wire Wire Line
 	1000 3100 1000 3300
 $Comp
-L NPN Q?
+L NPN Q11
 U 1 1 563C0D0A
 P 1400 5400
-F 0 "Q?" H 1400 5250 50  0000 R CNN
+F 0 "Q11" H 1400 5250 50  0000 R CNN
 F 1 "NPN" H 1400 5550 50  0000 R CNN
 F 2 "~" H 1400 5400 60  0000 C CNN
@@
 $EndComp
 $Comp
-L R R?
+L R R21
 U 1 1 563C0D0B
 P 1950 5400
-F 0 "R?" V 2030 5400 40  0000 C CNN
+F 0 "R21" V 2030 5400 40  0000 C CNN
 F 1 "10K" V 1957 5401 40  0000 C CNN
 F 2 "~" V 1880 5400 30  0000 C CNN
@@
 	1300 5200 1200 5200
 $Comp
-L GND #PWR?
+L GND #PWR28
 U 1 1 563C0D0C
 P 1300 5700
-F 0 "#PWR?" H 1300 5700 30  0001 C CNN
+F 0 "#PWR28" H 1300 5700 30  0001 C CNN
 F 1 "GND" H 1300 5630 30  0001 C CNN
 F 2 "" H 1300 5700 60  0000 C CNN
@@
 	2500 3500 3050 3500
 $Comp
-L NPN Q?
+L NPN Q12
 U 1 1 563C0D0D
 P 1400 7000
-F 0 "Q?" H 1400 6850 50  0000 R CNN
+F 0 "Q12" H 1400 6850 50  0000 R CNN
 F 1 "NPN" H 1400 7150 50  0000 R CNN
 F 2 "~" H 1400 7000 60  0000 C CNN
@@
 $EndComp
 $Comp
-L R R?
+L R R22
 U 1 1 563C0D0E
 P 1950 7000
-F 0 "R?" V 2030 7000 40  0000 C CNN
+F 0 "R22" V 2030 7000 40  0000 C CNN
 F 1 "10K" V 1957 7001 40  0000 C CNN
 F 2 "~" V 1880 7000 30  0000 C CNN
@@
 	1300 6800 1200 6800
 $Comp
-L GND #PWR?
+L GND #PWR29
 U 1 1 563C0D0F
 P 1300 7300
-F 0 "#PWR?" H 1300 7300 30  0001 C CNN
+F 0 "#PWR29" H 1300 7300 30  0001 C CNN
 F 1 "GND" H 1300 7230 30  0001 C CNN
 F 2 "" H 1300 7300 60  0000 C CNN
@@
 	2300 7000 2200 7000
 $Comp
-L 74HC04 U?
+L 74HC04 U5
 U 1 1 563C0D10
 P 2250 4500
-F 0 "U?" H 2400 4600 40  0000 C CNN
+F 0 "U5" H 2400 4600 40  0000 C CNN
 F 1 "74HC04" H 2450 4400 40  0000 C CNN
 F 2 "~" H 2250 4500 60  0000 C CNN
@@
 $EndComp
 $Comp
-L 74HC04 U?
-U 1 1 563C0D11
+L 74HC04 U5
+U 2 1 563C0D11
 P 2250 4900
-F 0 "U?" H 2400 5000 40  0000 C CNN
+F 0 "U5" H 2400 5000 40  0000 C CNN
 F 1 "74HC04" H 2450 4800 40  0000 C CNN
 F 2 "~" H 2250 4900 60  0000 C CNN
 F 3 "~" H 2250 4900 60  0000 C CNN
-	1    2250 4900
+	2    2250 4900
 	1    0    0    -1
 $EndComp
@@
 	1700 5400 1600 5400
 $Comp
-L R R?
+L R R19
 U 1 1 563C0D12
 P 1550 6700
-F 0 "R?" V 1630 6700 40  0000 C CNN
+F 0 "R19" V 1630 6700 40  0000 C CNN
 F 1 "10K" V 1557 6701 40  0000 C CNN
 F 2 "~" V 1480 6700 30  0000 C CNN
@@
 	1300 6700 1300 6800
 $Comp
-L 74HC04 U?
-U 1 1 563C0D13
+L 74HC04 U5
+U 4 1 563C0D13
 P 2250 6500
-F 0 "U?" H 2400 6600 40  0000 C CNN
+F 0 "U5" H 2400 6600 40  0000 C CNN
 F 1 "74HC04" H 2450 6400 40  0000 C CNN
 F 2 "~" H 2250 6500 60  0000 C CNN
 F 3 "~" H 2250 6500 60  0000 C CNN
-	1    2250 6500
+	4    2250 6500
 	1    0    0    -1
 $EndComp
@@
 	1800 6700 1800 6500
 $Comp
-L 74HC04 U?
-U 1 1 563C0D14
+L 74HC04 U5
+U 3 1 563C0D14
 P 2250 6100
-F 0 "U?" H 2400 6200 40  0000 C CNN
+F 0 "U5" H 2400 6200 40  0000 C CNN
 F 1 "74HC04" H 2450 6000 40  0000 C CNN
 F 2 "~" H 2250 6100 60  0000 C CNN
 F 3 "~" H 2250 6100 60  0000 C CNN
-	1    2250 6100
+	3    2250 6100
 	1    0    0    -1
 $EndComp
@@
 Wire Wire Line
 	1300 5100 1300 5200
-Text GLabel 5100 6150 2    60   Input ~ 0
-Pots_~SHDN~
-Text GLabel 5100 5350 2    60   Input ~ 0
-WATCHDOG
-Text GLabel 5100 6950 2    60   Input ~ 0
-Motor_Disable
 Text Notes 3900 4950 0    60   ~ 0
 Enable the Watchdog timer to force a Shutdown/Estop
@@
 	2800 6500 2700 6500
 $Comp
-L GS3 GS?
+L GS3 GS4
 U 1 1 563C0D15
 P 4750 5350
-F 0 "GS?" H 4800 5550 50  0000 C CNN
+F 0 "GS4" H 4800 5550 50  0000 C CNN
 F 1 "WD_select" H 4800 5151 40  0000 C CNN
 F 2 "GS3" V 4838 5276 30  0000 C CNN
@@
 $EndComp
 Wire Wire Line
-	5100 5350 4900 5350
+	5650 5350 4900 5350
 Wire Wire Line
 	4600 5250 4400 5250
@@
 	4600 5450 4400 5450
 $Comp
-L GS3 GS?
+L GS3 GS5
 U 1 1 563C0D16
 P 4750 6150
-F 0 "GS?" H 4800 6350 50  0000 C CNN
+F 0 "GS5" H 4800 6350 50  0000 C CNN
 F 1 "POT_select" H 4800 5951 40  0000 C CNN
 F 2 "GS3" V 4838 6076 30  0000 C CNN
@@
 $EndComp
 $Comp
-L GS3 GS?
+L GS3 GS6
 U 1 1 563C0D17
 P 4750 6950
-F 0 "GS?" H 4800 7150 50  0000 C CNN
+F 0 "GS6" H 4800 7150 50  0000 C CNN
 F 1 "INH_select" H 4800 6751 40  0000 C CNN
 F 2 "GS3" V 4838 6876 30  0000 C CNN
@@
 Text HLabel 3050 3500 2    60   Input ~ 0
 WATCHDOG_Pulse
+Text Label 5650 5350 2    60   ~ 0
+WATCHDOG
+Text HLabel 5100 6150 2    60   Input ~ 0
+Pots_~SHDN~
+Text Label 1000 3100 2    60   ~ 0
+WATCHDOG
+Text HLabel 5100 6950 2    60   Input ~ 0
+Motor_Disable
 $EndSCHEMATC
